Commit message: add datashow

File: workspace1/src/mrobot_gazebo/urdf/mrobot_body.urdf.xacro (robot description, xacro)
@@ -118,5 +118,5 @@
         </link>
         <gazebo reference="${fb}_caster_link">
-            <material>Gazebo/Black</material>
+            <material>Gazebo/Red</material>
         </gazebo>
         <joint name="base_to_${fb}_caster_joint" type="fixed">

File: workspace1/src/mrobot_gazebo/urdf/mrobot_with_sick_tim571.urdf.xacro (robot description, xacro)
@@ -9,5 +9,5 @@
 	<mrobot_body/>
 	<!-- Attach the Kinect -->
-	<joint name="rplidar_joint" type="fixed">
+	<joint name="sicktim571_joint" type="fixed">
 		<origin xyz="${rplidar_offset_x} ${rplidar_offset_y} ${rplidar_offset_z}" rpy="0 0 0" />
 		<parent link="plate_2_link"/>
